File: pogostick/pogostick.kicad_pcb (KiCad board)
At the start: 2 copper layers, 210 x 40 mm, 65 parts, among them J1 Pogo pin, J10 Pogo pin, J11 Pogo pin, J12 Pogo pin, J13 Pogo pin, J14 Pogo pin, J15 Pogo pin, J16 Pogo pin, J17 Pogo pin, J18 Pogo pin, J19 Pogo pin, J2 Pogo pin, J20 Pogo pin, J21 Pogo pin, J22 Pogo pin, J23 Pogo pin, J24 Pogo pin, J25 Pogo pin, J26 Pogo pin, J27 Pogo pin, J28 Pogo pin, J29 Pogo pin, J3 Pogo pin, J30 Pogo pin, J31 Pogo pin, J32 Pogo pin, J33 Pogo pin, J34 Pogo pin, J35 Pogo pin, J36 Pogo pin, J37 Pogo pin, J38 Pogo pin, J39 Pogo pin, J4 Pogo pin, J40 Pogo pin, J41 Pogo pin, J42 Pogo pin, J43 Pogo pin, J44 Pogo pin, J45 Pogo pin, J46 Pogo pin, J47 Pogo pin, J48 Pogo pin, J49 Pogo pin, J5 Pogo pin, J50 Pogo pin, J51 Pogo pin, J52 Pogo pin, J53 Pogo pin, J54 Pogo pin, J55 Pogo pin, J56 Pogo pin, J57 Pogo pin, J58 Pogo pin, J59 Pogo pin, J6 Pogo pin, J60 Pogo pin, J7 Pogo pin, J8 Pogo pin, J9 Pogo pin

Commit message: Add top pour for thermals and regenerate gerbers
Routing:
- added copper zone on F.Cu, net (none)

Commit message: Add more images of board
Parts:
- H3, H4, H5: footprint MountingHole:MountingHole_3.2mm_M3 -> MountingHole:MountingHole_3.2mm_M3_ISO7380_Pad_TopBottom
- moved H1 69.3 mm to (48.4, 54.0)
- moved H3 69.3 mm to (48.4, 74.0)
- moved H2 69.3 mm to (248.4, 54.0)
- moved H4 69.3 mm to (248.4, 74.0)
- moved H5 69.3 mm to (148.4, 84.0)
- moved J10 68.8 mm to (86.1, 67.0)
- moved J11 68.8 mm to (89.1, 67.0)
- moved J12 68.8 mm to (92.1, 67.0)
- moved J13 68.8 mm to (95.1, 67.0)
- moved J14 68.8 mm to (98.1, 67.0)
- moved J15 68.8 mm to (101.1, 67.0)
- moved J16 68.8 mm to (104.1, 67.0)
- moved J17 68.8 mm to (107.1, 67.0)
- moved J18 68.8 mm to (110.1, 67.0)
- moved J19 68.8 mm to (113.1, 67.0)
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Other:
- outline, holes or cut-outs redrawn
- board text added: "PHOTARA Pogo Pin Connector September 2026 Designed by Finn Hittson"
- board text removed: "Photara Pogo Pin Solar Cell Tester Board September 2026 Designed by Finn Hittson"
